File: z80.kicad_pcb (KiCad board)
At the start: 2 copper layers, 304.8 x 243.8 mm, 1 part

Commit message: Added some work to Z80 Address Bus and PCB
Parts:
- added DB-15: DSUB-15_Male_Horizontal_P2.77x2.84mm_EdgePinOffset4.94mm_Ho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, Connector_Dsub:DSUB-15_Male_Horizontal_P2.77x2.84mm_EdgePinOffset4.94mm_Housed_MountingHolesOffset7.48mm, F.Cu at (-1028.7, -843.3)
- added DB-25: DSUB-25_Female_Horizontal_P2.77x2.84mm_EdgePinOffset4.94mm_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, Connector_Dsub:DSUB-25_Female_Horizontal_P2.77x2.84mm_EdgePinOffset4.94mm_Housed_MountingHolesOffset7.48mm, F.Cu at (-951.2, -843.3)
- added DB9: DSUB-9_Female_Horizontal_P2.77x2.84mm_EdgePinOffset4.94mm_H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, Connector_Dsub:DSUB-9_Female_Horizontal_P2.77x2.84mm_EdgePinOffset4.94mm_Housed_MountingHolesOffset7.48mm, F.Cu at (-1052.8, -843.3)
- added REF**: MountingHole_2.2mm_M2_Pad_Via, MountingHole:MountingHole_2.2mm_M2_Pad_Via, F.Cu at (-876.3, -1004.6)
- added REF**: BatteryHolder_Keystone_103_1x20mm, Battery:BatteryHolder_Keystone_103_1x20mm, F.Cu at (-806.5, -852.2)
- added REF**: MountingHole_2.2mm_M2_Pad_Via, MountingHole:MountingHole_2.2mm_M2_Pad_Via, F.Cu at (-922.0, -1003.3)
- added REF**: MountingHole_2.2mm_M2_Pad_Via, MountingHole:MountingHole_2.2mm_M2_Pad_Via, F.Cu at (-961.4, -1003.3)
- added REF**: MountingHole_2.2mm_M2_Pad_Via, MountingHole:MountingHole_2.2mm_M2_Pad_Via, F.Cu at (-877.6, -1028.7)
- added REF**: MountingHole_2.2mm_M2_Pad_Via, MountingHole:MountingHole_2.2mm_M2_Pad_Via, F.Cu at (-878.8, -1050.3)
- added REF**: MountingHole_2.2mm_M2_Pad_Via, MountingHole:MountingHole_2.2mm_M2_Pad_Via, F.Cu at (-923.3, -1028.7)
- added REF**: MountingHole_2.2mm_M2_Pad_Via, MountingHole:MountingHole_2.2mm_M2_Pad_Via, F.Cu at (-924.6, -1050.3)
- added REF**: MountingHole_2.2mm_M2_Pad_Via, MountingHole:MountingHole_2.2mm_M2_Pad_Via, F.Cu at (-961.4, -1028.7)
- added REF**: MountingHole_2.2mm_M2_Pad_Via, MountingHole:MountingHole_2.2mm_M2_Pad_Via, F.Cu at (-1066.8, -1068.1)
- U1 Z80-CPU: renamed from REF**
- moved U1 Z80-CPU 206.4 mm to (-814.1, -1063.0)

Commit message: Added many components.
Parts:
- added U14: 74LS393, Package_DIP:DIP-14_W7.62mm_Socket, F.Cu at (-1016.0, -939.8)
- added U24: 74LS154, Package_DIP:DIP-24_W15.24mm_Socket, F.Cu at (-1038.9, -939.8)
- added U25: DIP-28_W15.24mm, Package_DIP:DIP-28_W15.24mm, F.Cu at (-991.9, -939.8)
- added U26: DIP-28_W15.24mm, Package_DIP:DIP-28_W15.24mm, F.Cu at (-971.5, -939.8)
