File: z80.sch (KiCad schematic (older format))
At the start: 67 parts

Commit message: Added some work to Z80 Address Bus and PCB
Parts:
- added C? (x3): CP, symbol Device:CP
- added J?: DB9_Female, symbol Connector:DB9_Female
- added JP1: Jumper, symbol Device:Jumper
- added R3, R4: 4k7, symbol Device:R
- added unit 1 of U3
- added unit 3 of U3
- added U4, U?: 74LS32, symbol 74xx:74LS32
- added U? (x2): 74LS393, symbol 74xx:74LS393
- added U? (x3): 74LS04, symbol 74xx:74LS04
- added U?: NA555D, Package_SO:SOIC-8_3.9x4.9mm_P1.27mm, symbol Timer:NA555D
- added U? (x2): HM62256BLP, Package_DIP:DIP-28_W15.24mm, symbol Memory_RAM:HM62256BLP
- added U?: 74LS08, symbol 74xx:74LS08
- U9: renamed from U?; footprint (none) -> Package_DIP:DIP-22_W7.62mm
- gave numbers to parts that had none: 4
Connections:
- net labels added: AddressBus
- wire segments 31 -> 135
Other:
- moved on the sheet: D?, J?, R?, RN?, SW?, U1, U10, U3B, U5, U9, U?, U?A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

Commit message: Added many components.
Parts:
- removed R?: R_Small_US, symbol Device:R_Small_US
- added C? (x3): CP1_Small, symbol Device:CP1_Small
- added C?: CP, symbol Device:CP
- added D?: 1N4001, Diode_THT:D_DO-41_SOD81_P10.16mm_Horizontal, symbol Diode:1N4001
- added D?: LED, symbol Device:LED
- added D?: 1N4007, Diode_THT:D_DO-41_SOD81_P10.16mm_Horizontal, symbol Diode:1N4007
- added J?: Conn_01x02_Female, symbol Connector:Conn_01x02_Female
- added J? (x2): Conn_02x13_Odd_Even, symbol Connector_Generic:Conn_02x13_Odd_Even
- added Q?: BC547, Package_TO_SOT_THT:TO-92_Inline, symbol Transistor_BJT:BC547
- added Q?: BC557, Package_TO_SOT_THT:TO-92_Inline, symbol Transistor_BJT:BC557
- added R14, R17: 1K, symbol Device:R_Small
- added R? (x2): R_Small, symbol Device:R_Small
- added RN?: R_Network09_US, Resistor_THT:R_Array_SIP10, symbol Device:R_Network09_US
- added SW?: SW_Push, symbol Switch:SW_Push
- added U?: 74LS670, symbol 74xx:74LS670
- added U?: HM62256BLP, Package_DIP:DIP-28_W15.24mm, symbol Memory_RAM:HM62256BLP
- added U?: 27C128, Package_DIP:DIP-28_W15.24mm, symbol Memory_EPROM:27C128
- added U? (x2): 74LS123, symbol 74xx:74LS123
- added U?: LM7905_TO220, Package_TO_SOT_THT:TO-220-3_Vertical, symbol Regulator_Linear:LM7905_TO220
- added U?: TL7705A, symbol Power_Supervisor:TL7705A
- added U?: 74LS374, symbol 74xx:74LS374
- added U?: 74LS00, symbol 74xx:74LS00
- added U? (x2): 74LS373, symbol 74xx:74LS373
- added U? (x3): 74LS157, symbol 74xx:74LS157
- added U?: 74LS244, symbol 74xx:74LS244
- added U?: 74LS04, symbol 74xx:74LS04
- added U?: 74LS153, symbol 74xx:74LS153
- added U?: 74LS682, symbol 74xx_IEEE:74LS682
- added U?: 628128_TSOP32, symbol Memory_RAM:628128_TSOP32
- added U? (x4): 74LS14, symbol 74xx:74LS14
- added U?: 74LS90, symbol 74xx:74LS90
- added U?: GAL16V8, symbol Logic_Programmable:GAL16V8
- added Y1: Crystal, 3.579MHz, symbol Device:Crystal
- U1: value Z80CPU -> Z84C0008PEC
- gave numbers to parts that had none: 4
Connections:
- wire segments 135 -> 304
Other:
- note added: "CPU"
- note added: "Composite Video"
- moved on the sheet: C?, D?, J?, R?, SW?, U1, U10, U11A, U26, U5, U9, U?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
